File: accl_magn_pmod.kicad_sch (KiCad schematic)
At the start: 16 parts, among them J1 pmod, U1 adxl345, U2 hmc5883l

Commit message: add screenshots
Other:
- company: (none) -> S59MZ
- title: (none) -> accl-magn-pmod
